File: CJ4-Autopilot.kicad_pcb (KiCad board)
At the start: 2 copper layers, 154.8 x 93.1 mm, 46 parts, among them J1 Conn_01x05, J2 Conn_01x05, J3 Conn_01x05, J4 Conn_01x05, SW1 SW_Push_LED, SW10 SW_Push_LED, SW11 SW_Push_LED, SW12 SW_Push_LED, SW13 SW_Push_LED, SW14 SW_Push_LED, SW15 SW_Push, SW16 RotaryEncoder, SW2 SW_Push_LED, SW3 SW_Push_LED, SW4 SW_Push_LED, SW5 SW_Push_LED, SW6 SW_Push_LED, SW7 SW_Push_LED, SW8 SW_Push_LED, SW9 SW_Push_LED, U1 TLC5917IN, U2 Pico, U3 TLC5917IN, U4 74HC165, U5 74HC165

Commit message: Initial board layout, still a lot of work to do
Parts:
- added H12: MountingHole, CJ4-Autopilot:JLCPCB_Tooling_Hole, F.Cu at (24.1, 52.8)
- added J5: CRS encoder, Connector_JST:JST_XA_B05B-XASK-1_1x05_P2.50mm_Vertical, B.Cu at (299.7, 45.8)
- C1, C2, C3, C4, U1, U2, U3, U4, U5: moved to B.Cu
- H10, H11: footprint MountingHole:MountingHole_3.2mm_M3 -> CJ4-Autopilot:JLCPCB_Tooling_Hole
- H5: value MountingHole -> CRS1 encoder
- H6: value MountingHole -> FLC encoder
- H7: value MountingHole -> HDG encoder
- H8: value MountingHole -> ALT encoder
- H9: value MountingHole -> CRS2 encoder; footprint MountingHole:MountingHole_3.2mm_M3 -> CJ4-Autopilot:MountingHole_7.5mm
- J1: value Conn_01x05 -> CRS encoder; footprint CJ4-Autopilot:SW_PUSH_6mm -> Connector_JST:JST_XA_B05B-XASK-1_1x05_P2.50mm_Vertical; moved to B.Cu
- J2: value Conn_01x05 -> FLC encoder; footprint CJ4-Autopilot:SW_PUSH_6mm -> Connector_JST:JST_XA_B05B-XASK-1_1x05_P2.50mm_Vertical; moved to B.Cu
- J3: value Conn_01x05 -> HDG encoder; footprint CJ4-Autopilot:SW_PUSH_6mm -> Connector_JST:JST_XA_B05B-XASK-1_1x05_P2.50mm_Vertical; moved to B.Cu
- J4: value Conn_01x05 -> ALT encoder; footprint CJ4-Autopilot:SW_PUSH_6mm -> Connector_JST:JST_XA_B05B-XASK-1_1x05_P2.50mm_Vertical; moved to B.Cu
- R1, R2: footprint CJ4-Autopilot:SW_PUSH_6mm -> Resistor_SMD:R_0603_1608Metric; moved to B.Cu
- RN1, RN2, RN3, RN4: footprint CJ4-Autopilot:SW_PUSH_6mm -> Resistor_SMD:R_Array_Convex_4x0603; moved to B.Cu
- SW1: value SW_Push_LED -> FD1
- SW10: value SW_Push_LED -> ALT
- SW11: value SW_Push_LED -> YD
- SW12: value SW_Push_LED -> XFR
- SW13: value SW_Push_LED -> AP
- SW14: value SW_Push_LED -> FD2
- SW15: value SW_Push -> DISC
- SW16: value RotaryEncoder -> VS encoder
- SW2: value SW_Push_LED -> VS
- SW3: value SW_Push_LED -> VNAV
- SW4: value SW_Push_LED -> FLC
- SW5: value SW_Push_LED -> NAV
- SW6: value SW_Push_LED -> BANK
- SW7: value SW_Push_LED -> HDG
- SW8: value SW_Push_LED -> APPR
- SW9: value SW_Push_LED -> BC
- moved H2 208.7 mm to (331.5, 24.1)
- moved H9 191.9 mm to (311.1, 50.8)
- moved SW14 188.4 mm to (307.9, 29.5)
- moved U2 176.9 mm to (266.7, 99.1), turned to -90 degrees
- moved H4 169.5 mm to (331.5, 58.4)
- moved SW13 168.4 mm to (280.0, 29.5)
- moved H10 166.7 mm to (24.1, 29.3)
- moved SW15 164.3 mm to (280.0, 48.5)
- moved H1 157.5 mm to (24.1, 24.1)
- moved H11 157.0 mm to (331.5, 29.2)
- moved H3 132.1 mm to (24.1, 58.4)
- moved H8 127.0 mm to (233.7, 50.8)
- moved J3 124.6 mm to (189.9, 45.8), turned to -90 degrees
- moved C2 115.3 mm to (219.7, 21.0)
- moved C3 113.7 mm to (267.3, 37.3), turned to -90 degrees
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Connections:
- J2 pad 4: SPEED_BTN -> FLC_BTN
- J4 pad 1: CRS2_A -> ALT_A
- J4 pad 3: CRS2_B -> ALT_B
- J4 pad 4: CRS2_BTN -> ALT_BTN
- U1 pad 16: GND -> +3V3
- U2 pad 31: unconnected-(U2-Pad31) -> ALT_BTN
- U2 pad 32: unconnected-(U2-Pad32) -> ALT_B
- U2 pad 34: unconnected-(U2-Pad34) -> ALT_A
- U3 pad 16: GND -> +3V3
Routing:
- added copper zone on B.Cu, net GND
- added copper zone on F.Cu, net GND
Other:
- board size 154.8 x 93.1 mm -> 317.5 x 44.5 mm

Commit message: Add RP2040 directly to the board
Parts:
- added C10: 100nF, CJ4-Autopilot:Perfect_0402, B.Cu at (212.2, 92.4)
- added C11: 100nF, CJ4-Autopilot:Perfect_0402, B.Cu at (206.4, 86.1)
- added C12: 1uF, CJ4-Autopilot:Perfect_0402, B.Cu at (203.5, 88.1)
- added C13: 100nF, CJ4-Autopilot:Perfect_0402, B.Cu at (199.1, 84.0)
- added C14: 1uF, CJ4-Autopilot:Perfect_0402, B.Cu at (212.2, 94.4)
- added C15: 100nF, CJ4-Autopilot:Perfect_0402, B.Cu at (200.6, 82.1)
- added C16: 100nF, CJ4-Autopilot:Perfect_0402, B.Cu at (206.4, 88.1)
- added C17: 100nF, CJ4-Autopilot:Perfect_0402, B.Cu at (197.7, 82.1)
- added C18: 100nF, CJ4-Autopilot:Perfect_0402, B.Cu at (193.1, 74.9)
- added C19: 100nF, CJ4-Autopilot:Perfect_0402, B.Cu at (193.1, 78.8)
- added C20: 100nF, CJ4-Autopilot:Perfect_0402, B.Cu at (215.7, 81.1)
- added C5: 20pF, CJ4-Autopilot:Perfect_0402, B.Cu at (193.1, 76.8)
- added C6: 20pF, CJ4-Autopilot:Perfect_0402, B.Cu at (209.3, 92.4)
- added C7: 10uF, Capacitor_SMD:C_0603_1608Metric, B.Cu at (215.8, 92.9)
- added C8: 100nF, CJ4-Autopilot:Perfect_0402, B.Cu at (195.9, 74.9)
- added C9: 10uF, Capacitor_SMD:C_0603_1608Metric, B.Cu at (205.6, 83.6)
- added J6: USB_B_Micro, CJ4-Autopilot:USB_B_Mini_Amphenol_UE25BE5510H, B.Cu at (222.7, 91.9)
- added J7: Conn_01x02, Connector_PinHeader_2.54mm:PinHeader_1x02_P2.54mm_Vertical, B.Cu at (199.7, 76.2)
- added R3: 1k, CJ4-Autopilot:Perfect_0402, B.Cu at (201.9, 84.0)
- added R4: 1k, CJ4-Autopilot:Perfect_0402, B.Cu at (206.4, 90.1)
- added R5: DNF, Resistor_SMD:R_1206_3216Metric_Pad1.30x1.75mm_HandSolder, B.Cu at (189.2, 88.9)
- added R6: 27, Resistor_SMD:R_0603_1608Metric, B.Cu at (182.9, 75.6)
- added R7: 27, Resistor_SMD:R_0603_1608Metric, B.Cu at (187.3, 75.6)
- added U6: W25Q128JVS, Package_SO:SOIC-8_5.23x5.23mm_P1.27mm, B.Cu at (222.3, 83.5)
- added U7: RP2040, RP2040_minimal:RP2040-QFN-56, B.Cu at (212.5, 86.8)
- added Y1: X322512MSB4SI, Crystal:Crystal_SMD_3225-4Pin_3.2x2.5mm, B.Cu at (199.4, 102.9)
- J1, J2, J3, J4, J5: footprint Connector_JST:JST_XA_B05B-XASK-1_1x05_P2.50mm_Vertical -> Connector_JST:JST_XH_B5B-XH-A_1x05_P2.50mm_Vertical
- R1, R2: footprint Resistor_SMD:R_0603_1608Metric -> CJ4-Autopilot:Perfect_0402
- U1, U3: footprint Package_DIP:DIP-16_W7.62mm -> Package_SO:SOIC-16_3.9x9.9mm_P1.27mm
- U2: value Pico -> AMS1117-3.3; footprint MCU_RaspberryPi_and_Boards:RPi_Pico_SMD_TH -> CJ4-Autopilot:SOT-223-4NC
- moved RN2 90.8 mm to (58.4, 57.1), turned to -90 degrees
- moved RN4 85.1 mm to (58.4, 44.5), turned to -90 degrees
- moved R1 80.9 mm to (293.4, 36.8), turned to 180 degrees
- moved C4 79.5 mm to (52.1, 50.8)
- moved U5 78.1 mm to (58.4, 50.8), turned to -90 degrees
- moved U1 74.1 mm to (297.2, 31.8), turned to -90 degrees
- moved C2 71.9 mm to (290.8, 31.8), turned to 90 degrees
- moved R2 68.6 mm to (54.0, 36.8)
- moved C1 67.3 mm to (51.4, 31.6)
- moved U3 63.6 mm to (57.8, 31.8)
- moved U2 63.4 mm to (206.9, 78.0), turned to 180 degrees
- moved RN3 36.4 mm to (297.2, 44.5), turned to 90 degrees
- moved RN1 36.0 mm to (297.2, 57.1), turned to 90 degrees
- moved C3 27.1 mm to (290.8, 50.8)
- moved U4 26.5 mm to (297.2, 50.8), turned to -90 degrees
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Connections:
- SW1 pad 3: +5V -> VBUS
- SW10 pad 3: +5V -> VBUS
- SW11 pad 3: +5V -> VBUS
- SW12 pad 3: +5V -> VBUS
- SW13 pad 3: +5V -> VBUS
- SW14 pad 3: +5V -> VBUS
- SW2 pad 3: +5V -> VBUS
- SW3 pad 3: +5V -> VBUS
- SW4 pad 3: +5V -> VBUS
- SW5 pad 3: +5V -> VBUS
- SW6 pad 3: +5V -> VBUS
- SW7 pad 3: +5V -> VBUS
- SW8 pad 3: +5V -> VBUS
- SW9 pad 3: +5V -> VBUS
- U2 pad 1: unconnected-(U2-Pad1) -> GND
- U2 pad 2: unconnected-(U2-Pad2) -> +3V3
- U2 pad 3: GND -> VBUS
Other:
- outline, holes or cut-outs redrawn

Commit message: RP2040 wired up, warning cleanup
Parts:
- U2: footprint CJ4-Autopilot:SOT-223-4NC -> Package_TO_SOT_SMD:SOT-223-3_TabPin2
- moved C7 117.2 mm to (121.9, 22.9)
- moved J6 112.9 mm to (131.1, 25.9)
- moved C14 102.6 mm to (125.9, 38.9), turned to 90 degrees
- moved C20 100.3 mm to (123.4, 41.8)
- moved U2 98.4 mm to (121.7, 29.0), turned to -90 degrees
- moved C9 97.9 mm to (120.9, 34.5)
- moved C10 97.2 mm to (131.1, 38.9), turned to 90 degrees
- moved U6 96.4 mm to (138.4, 36.1)
- moved C16 92.1 mm to (123.8, 47.3)
- moved U7 92.0 mm to (130.0, 46.0)
- moved C12 90.9 mm to (127.1, 38.9), turned to 90 degrees
- moved C6 87.0 mm to (130.6, 55.3)
- moved C11 84.9 mm to (128.3, 52.7), turned to -90 degrees
- moved R4 83.6 mm to (131.3, 53.3), turned to -90 degrees
- moved C13 82.7 mm to (129.8, 38.9), turned to 90 degrees
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Routing:
- net VBUS: track 0.00 -> 385.8 mm
- net +3V3: track 0.00 -> 28.5 mm
- net GND: track 0.00 -> 27.1 mm, vias 0 -> 22
- net /RP2040/QSPI_SS: track 0.00 -> 21.4 mm
- net +1V1: track 0.00 -> 18.7 mm, vias 0 -> 4
- net /RP2040/QSPI_SD1: track 0.00 -> 17.7 mm
- net /RP2040/QSPI_SD2: track 0.00 -> 13.2 mm
- net /RP2040/XIN: track 0.00 -> 11.0 mm
- net /RP2040/QSPI_SD3: track 0.00 -> 8.94 mm
- net /RP2040/QSPI_SCLK: track 0.00 -> 7.51 mm
- net Net-(R7-Pad2): track 0.00 -> 6.72 mm
- net Net-(R6-Pad2): track 0.00 -> 6.32 mm
- net /RP2040/QSPI_SD0: track 0.00 -> 5.97 mm
- net /RP2040/~{USB_BOOT}: track 0.00 -> 5.71 mm
- net /RP2040/XOUT: track 0.00 -> 3.86 mm
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- added copper zone on B.Cu, net +1V1
- added copper zone on B.Cu, net +3V3
- added copper zone on B.Cu, net VBUS
Other:
- board size 317.5 x 44.5 mm -> 317.5 x 50.8 mm

Commit message: Update encoder footprint, USB trace width
Parts:
- H5, H6, H7, H8, H9: footprint CJ4-Autopilot:MountingHole_7.5mm -> CJ4-Autopilot:EN11-HSM1BF20 panel mount
Routing:
- net /RP2040/USB_D+: track 0.00 -> 12.5 mm
- net /RP2040/USB_D-: track 0.00 -> 8.60 mm
Changed lines of the file:
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@@
       (solder_mask_margin 0.148))
   )
-  (footprint "CJ4-Autopilot:MountingHole_7.5mm" (layer "F.Cu")
+  (footprint "CJ4-Autopilot:EN11-HSM1BF20 panel mount" (layer "F.Cu")
     (at 233.68 50.8)
-    (descr "Mounting Hole 7.5mm, no annular")
-    (tags "mounting hole 7.5mm no annular")
+    (descr "EN11-HSM1BF20 panel mount")
+    (tags "EN11-HSM1BF20")
     (property "Sheetfile" "CJ4-Autopilot.kicad_sch")
     (property "Sheetname" "")
@@
       (effects (font (size 1 1) (thickness 0.15)))
     )
-    (fp_text value "ALT encoder" (at 0 7) (layer "F.Fab")
+    (fp_text value "ALT encoder" (at 0 8.001) (layer "F.Fab")
       (effects (font (size 1 1) (thickness 0.15)))
     )
@@
     )
     (fp_circle (center 0 0) (end 6 0) (layer "Cmts.User") (width 0.15) (fill none))
-    (fp_circle (center 0 0) (end 6.25 0) (layer "F.CrtYd") (width 0.05) (fill none))
+    (fp_line (start 1.586121 6.858) (end -1.524 6.858) (layer "F.CrtYd") (width 0.05))
+    (fp_line (start -1.524 6.095999) (end -1.524 6.858) (layer "F.CrtYd") (width 0.05))
+    (fp_line (start 1.586121 6.858) (end 1.586121 6.080132) (layer "F.CrtYd") (width 0.05))
+    (fp_arc (start -1.524 6.095999) (mid -0.032056 -6.28353) (end 1.586121 6.080132) (layer "F.CrtYd") (width 0.05))
+    (pad "" np_thru_hole rect (at 0 6 90) (size 1 2.2) (drill oval 0.9 2.1) (layers F&B.Cu *.Mask))
     (pad "" np_thru_hole circle (at 0 0) (size 7.5 7.5) (drill 7.5) (layers F&B.Cu *.Mask))
-    (model "${KIPRJMOD}/3D Models/EN11-HSM1BF20--3DModel-STEP-412949.STEP"
-      (offset (xyz 0 0 -1.905))
-      (scale (xyz 1 1 1))
-      (rotate (xyz -90 0 0))
-    )
   )
   (footprint "CJ4-Autopilot:SW_PUSH_6mm" (layer "F.Cu")
@@
     )
   )
-  (footprint "CJ4-Autopilot:MountingHole_7.5mm" (layer "F.Cu")
+  (footprint "CJ4-Autopilot:EN11-HSM1BF20 panel mount" (layer "F.Cu")
     (at 311.15 50.8)
-    (descr "Mounting Hole 7.5mm, no annular")
-    (tags "mounting hole 7.5mm no annular")
+    (descr "EN11-HSM1BF20 panel mount")
+    (tags "EN11-HSM1BF20")
     (property "Sheetfile" "CJ4-Autopilot.kicad_sch")
     (property "Sheetname" "")
@@
       (effects (font (size 1 1) (thickness 0.15)))
     )
-    (fp_text value "CRS2 encoder" (at 0 7) (layer "F.Fab")
+    (fp_text value "CRS2 encoder" (at 0 8.001) (layer "F.Fab")
       (effects (font (size 1 1) (thickness 0.15)))
     )
@@
     )
     (fp_circle (center 0 0) (end 6 0) (layer "Cmts.User") (width 0.15) (fill none))
-    (fp_circle (center 0 0) (end 6.25 0) (layer "F.CrtYd") (width 0.05) (fill none))
+    (fp_line (start -1.524 6.095999) (end -1.524 6.858) (layer "F.CrtYd") (width 0.05))
+    (fp_line (start 1.586121 6.858) (end 1.586121 6.080132) (layer "F.CrtYd") (width 0.05))
+    (fp_line (start 1.586121 6.858) (end -1.524 6.858) (layer "F.CrtYd") (width 0.05))
+    (fp_arc (start -1.524 6.095999) (mid -0.032056 -6.28353) (end 1.586121 6.080132) (layer "F.CrtYd") (width 0.05))
+    (pad "" np_thru_hole rect (at 0 6 90) (size 1 2.2) (drill oval 0.9 2.1) (layers F&B.Cu *.Mask))
     (pad "" np_thru_hole circle (at 0 0) (size 7.5 7.5) (drill 7.5) (layers F&B.Cu *.Mask))
-    (model "${KIPRJMOD}/3D Models/EN11-HSM1BF20--3DModel-STEP-412949.STEP"
-      (offset (xyz 0 0 -1.905))
-      (scale (xyz 1 1 1))
-      (rotate (xyz -90 0 0))
-    )
   )
   (footprint "CJ4-Autopilot:SW_PUSH_6mm" (layer "F.Cu")
@@
     )
   )
-  (footprint "CJ4-Autopilot:MountingHole_7.5mm" (layer "F.Cu")
+  (footprint "CJ4-Autopilot:EN11-HSM1BF20 panel mount" (layer "F.Cu")
     (at 177.8 50.8)
-    (descr "Mounting Hole 7.5mm, no annular")
-    (tags "mounting hole 7.5mm no annular")
+    (descr "EN11-HSM1BF20 panel mount")
+    (tags "EN11-HSM1BF20")
     (property "Sheetfile" "CJ4-Autopilot.kicad_sch")
     (property "Sheetname" "")
@@
       (effects (font (size 1 1) (thickness 0.15)))
     )
-    (fp_text value "HDG encoder" (at 0 7) (layer "F.Fab")
+    (fp_text value "HDG encoder" (at 0 8.001) (layer "F.Fab")
       (effects (font (size 1 1) (thickness 0.15)))
     )
@@
     )
     (fp_circle (center 0 0) (end 6 0) (layer "Cmts.User") (width 0.15) (fill none))
-    (fp_circle (center 0 0) (end 6.25 0) (layer "F.CrtYd") (width 0.05) (fill none))
+    (fp_line (start -1.524 6.095999) (end -1.524 6.858) (layer "F.CrtYd") (width 0.05))
+    (fp_line (start 1.586121 6.858) (end -1.524 6.858) (layer "F.CrtYd") (width 0.05))
+    (fp_line (start 1.586121 6.858) (end 1.586121 6.080132) (layer "F.CrtYd") (width 0.05))
+    (fp_arc (start -1.524 6.095999) (mid -0.032056 -6.28353) (end 1.586121 6.080132) (layer "F.CrtYd") (width 0.05))
     (pad "" np_thru_hole circle (at 0 0) (size 7.5 7.5) (drill 7.5) (layers F&B.Cu *.Mask))
-    (model "${KIPRJMOD}/3D Models/EN11-HSM1BF20--3DModel-STEP-412949.STEP"
-      (offset (xyz 0 0 -1.905))
-      (scale (xyz 1 1 1))
-      (rotate (xyz -90 0 0))
-    )
+    (pad "" np_thru_hole rect (at 0 6 90) (size 1 2.2) (drill oval 0.9 2.1) (layers F&B.Cu *.Mask))
   )
   (footprint "MountingHole:MountingHole_3.2mm_M3" (layer "F.Cu")
@@
     (pad "" np_thru_hole circle (at 0 0) (size 3.2 3.2) (drill 3.2) (layers *.Cu *.Mask))
   )
-  (footprint "CJ4-Autopilot:MountingHole_7.5mm" (layer "F.Cu")
+  (footprint "CJ4-Autopilot:EN11-HSM1BF20 panel mount" (layer "F.Cu")
     (at 111.76 50.8)
-    (descr "Mounting Hole 7.5mm, no annular")
-    (tags "mounting hole 7.5mm no annular")
+    (descr "EN11-HSM1BF20 panel mount")
+    (tags "EN11-HSM1BF20")
     (property "Sheetfile" "CJ4-Autopilot.kicad_sch")
     (property "Sheetname" "")
@@
       (effects (font (size 1 1) (thickness 0.15)))
     )
-    (fp_text value "FLC encoder" (at 0 7) (layer "F.Fab")
+    (fp_text value "FLC encoder" (at 0 8.001) (layer "F.Fab")
       (effects (font (size 1 1) (thickness 0.15)))
     )
@@
     )
     (fp_circle (center 0 0) (end 6 0) (layer "Cmts.User") (width 0.15) (fill none))
-    (fp_circle (center 0 0) (end 6.25 0) (layer "F.CrtYd") (width 0.05) (fill none))
+    (fp_line (start 1.586121 6.858) (end 1.586121 6.080132) (layer "F.CrtYd") (width 0.05))
+    (fp_line (start 1.586121 6.858) (end -1.524 6.858) (layer "F.CrtYd") (width 0.05))
+    (fp_line (start -1.524 6.095999) (end -1.524 6.858) (layer "F.CrtYd") (width 0.05))
+    (fp_arc (start -1.524 6.095999) (mid -0.032056 -6.28353) (end 1.586121 6.080132) (layer "F.CrtYd") (width 0.05))
     (pad "" np_thru_hole circle (at 0 0) (size 7.5 7.5) (drill 7.5) (layers F&B.Cu *.Mask))
-    (model "${KIPRJMOD}/3D Models/EN11-HSM1BF20--3DModel-STEP-412949.STEP"
-      (offset (xyz 0 0 -1.905))
-      (scale (xyz 1 1 1))
-      (rotate (xyz -90 0 0))
-    )
+    (pad "" np_thru_hole rect (at 0 6 90) (size 1 2.2) (drill oval 0.9 2.1) (layers F&B.Cu *.Mask))
   )
   (footprint "CJ4-Autopilot:SW_PUSH_6mm" (layer "F.Cu")
@@
     )
   )
-  (footprint "CJ4-Autopilot:MountingHole_7.5mm" (layer "F.Cu")
+  (footprint "CJ4-Autopilot:EN11-HSM1BF20 panel mount" (layer "F.Cu")
     (at 44.45 50.8)
-    (descr "Mounting Hole 7.5mm, no annular")
-    (tags "mounting hole 7.5mm no annular")
+    (descr "EN11-HSM1BF20 panel mount")
+    (tags "EN11-HSM1BF20")
     (property "Sheetfile" "CJ4-Autopilot.kicad_sch")
     (property "Sheetname" "")
@@
       (effects (font (size 1 1) (thickness 0.15)))
     )
-    (fp_text value "CRS1 encoder" (at 0 7) (layer "F.Fab")
+    (fp_text value "CRS1 encoder" (at 0 8.001) (layer "F.Fab")
       (effects (font (size 1 1) (thickness 0.15)))
     )
@@
     )
     (fp_circle (center 0 0) (end 6 0) (layer "Cmts.User") (width 0.15) (fill none))
-    (fp_circle (center 0 0) (end 6.25 0) (layer "F.CrtYd") (width 0.05) (fill none))
+    (fp_line (start -1.524 6.095999) (end -1.524 6.858) (layer "F.CrtYd") (width 0.05))
+    (fp_line (start 1.586121 6.858) (end 1.586121 6.080132) (layer "F.CrtYd") (width 0.05))
+    (fp_line (start 1.586121 6.858) (end -1.524 6.858) (layer "F.CrtYd") (width 0.05))
+    (fp_arc (start -1.524 6.095999) (mid -0.032056 -6.28353) (end 1.586121 6.080132) (layer "F.CrtYd") (width 0.05))
     (pad "" np_thru_hole circle (at 0 0) (size 7.5 7.5) (drill 7.5) (layers F&B.Cu *.Mask))
-    (model "${KIPRJMOD}/3D Models/EN11-HSM1BF20--3DModel-STEP-412949.STEP"
-      (offset (xyz 0 0 -1.905))
-      (scale (xyz 1 1 1))
-      (rotate (xyz -90 0 0))
-    )
+    (pad "" np_thru_hole rect (at 0 6 90) (size 1 2.2) (drill oval 0.9 2.1) (layers F&B.Cu *.Mask))
   )
   (footprint "CJ4-Autopilot:SW_PUSH_6mm" (layer "F.Cu")
@@
   (segment (start 129.448 50.871205) (end 129.2485 51.070705) (width 0.2) (layer "B.Cu") (net 59))
   (segment (start 130.248 40.567) (end 130.248 40.44) (width 0.2) (layer "B.Cu") (net 59))
+  (segment (start 133.083176 26.67) (end 133.096 26.67) (width 0.4) (layer "B.Cu") (net 61))
+  (segment (start 131.064 24.608) (end 131.064 24.650824) (width 0.4) (layer "B.Cu") (net 61))
+  (segment (start 133.096 27.901666) (end 133.096 26.67) (width 0.8) (layer "B.Cu") (net 61))
+  (segment (start 129.159 34.616) (end 129.159 31.838666) (width 0.8) (layer "B.Cu") (net 61))
+  (segment (start 129.159 31.838666) (end 133.096 27.901666) (width 0.8) (layer "B.Cu") (net 61))
+  (segment (start 131.064 24.650824) (end 133.083176 26.67) (width 0.4) (layer "B.Cu") (net 61))
+  (segment (start 127.381 34.616) (end 127.381 31.623) (width 0.8) (layer "B.Cu") (net 62))
+  (segment (start 127.381 31.623) (end 130.264 28.74) (width 0.8) (layer "B.Cu") (net 62))
+  (segment (start 130.264 28.74) (end 130.264 27.208) (width 0.8) (layer "B.Cu") (net 62))
   (segment (start 139.827 30.488) (end 139.827 26.04) (width 0.25) (layer "B.Cu") (net 63))
   (segment (start 139.827 26.04) (end 138.933 25.146) (width 0.25) (layer "B.Cu") (net 63))
