File: CJ4-Autopilot.kicad_pcb (KiCad board)
At the start: 2 copper layers, 317.5 x 50.8 mm, 76 parts, among them J1 CRS encoder, J2 FLC encoder, J3 HDG encoder, J4 ALT encoder, J5 CRS encoder, J6 USB_B_Micro, J7 Conn_01x02, SW1 FD1, SW10 ALT, SW11 YD, SW12 XFR, SW13 AP, SW14 FD2, SW15 DISC, SW16 VS encoder, SW2 VS, SW3 VNAV, SW4 FLC, SW5 NAV, SW6 BANK, SW7 HDG, SW8 APPR, SW9 BC, U1 TLC5917IN, U2 AMS1117-3.3, U3 TLC5917IN, U4 74HC165, U5 74HC165, U6 W25Q128JVS, U7 RP2040, Y1 X322512MSB4SI

Commit message: Tons and tons of traces
Parts:
- moved C2 52.7 mm to (254.2, 49.1)
- moved U3 52.7 mm to (247.9, 50.5)
- moved R2 52.7 mm to (251.7, 46.0)
- moved C4 30.2 mm to (197.8, 38.7)
- moved RN1 30.2 mm to (190.9, 33.7)
- moved RN2 30.2 mm to (190.9, 48.1)
- moved U4 30.2 mm to (190.9, 41.5)
- moved C1 15.7 mm to (171.0, 44.2)
- moved U1 15.6 mm to (162.8, 47.2)
- moved R1 15.6 mm to (166.4, 42.7)
- moved C3 9.40 mm to (304.3, 38.4)
- moved RN3 9.40 mm to (297.2, 35.1), turned to -90 degrees
- moved RN4 9.40 mm to (296.9, 48.0)
- moved U5 9.40 mm to (297.2, 41.1)
Connections:
- RN1 pad 5: /Input shifter/D3 -> APPR
- RN1 pad 7: /Input shifter/D1 -> HDG
- RN1 pad 8: /Input shifter/D0 -> NAV
- RN2 pad 5: HDG -> BANK
- RN2 pad 6: HDG -> /Input shifter/D6
- RN2 pad 7: BANK -> /Input shifter/D5
- RN2 pad 8: NAV -> BC
- RN3 pad 8: BC -> /Input shifter1/D0
- RN4 pad 5: DISC -> /Input shifter1/D7
- U1 pad 10: VNAV_LED -> NAV_LED
- U1 pad 11: VS_LED -> HDG_LED
- U1 pad 12: FLC_LED -> unconnected-(U1-Pad12)
- U1 pad 5: NAV_LED -> FD1_LED
- U1 pad 6: BANK_LED -> VNAV_LED
- U1 pad 7: HDG_LED -> VS_LED
- U1 pad 8: APPR_LED -> FLC_LED
- U1 pad 9: FD1_LED -> BANK_LED
- U3 pad 11: unconnected-(U3-Pad11) -> AP_LED
- U3 pad 5: BC_LED -> XFR_LED
- U3 pad 6: ALT_LED -> BC_LED
- U3 pad 7: YD_LED -> APPR_LED
- U3 pad 8: XFR_LED -> ALT_LED
- U3 pad 9: AP_LED -> YD_LED
- U4 pad 11: /Input shifter/D0 -> NAV
- U4 pad 12: /Input shifter/D1 -> HDG
- U4 pad 14: /Input shifter/D3 -> APPR
- U4 pad 3: NAV -> BC
- U4 pad 4: BANK -> /Input shifter/D5
- U4 pad 5: HDG -> /Input shifter/D6
- U4 pad 6: APPR -> BANK
- U5 pad 11: BC -> /Input shifter1/D0
- U7 pad 11: SPEED_BTN -> LED_LATCH
- U7 pad 4: /RP2040/GPIO02 -> BTN_DATA
- U7 pad 5: /RP2040/GPIO03 -> BTN_LATCH
- U7 pad 6: LED_CLOCK -> BTN_CLOCK
- U7 pad 7: LED_LATCH -> BACKLIGHT_BRIGHT
- U7 pad 8: /RP2040/GPIO06 -> LED_DATA
- U7 pad 9: LED_DATA -> LED_CLOCK
Routing:
- net BTN_LATCH: track 0.00 -> 172.1 mm
- net BTN_CLOCK: track 0.00 -> 172.0 mm
- net BTN_DATA: track 0.00 -> 161.7 mm
- net BACKLIGHT_BRIGHT: track 0.00 -> 134.2 mm, vias 0 -> 2
- net LED_LATCH: track 0.00 -> 132.9 mm
- net LED_CLOCK: track 0.00 -> 131.0 mm, vias 0 -> 2
- net /Input shifter/QH: track 0.00 -> 109.7 mm
- net /SDO: track 0.00 -> 103.5 mm, vias 0 -> 2
- net FD2_LED: track 0.00 -> 78.9 mm, vias 0 -> 4
- net APPR_LED: track 0.00 -> 52.5 mm, vias 0 -> 2
- net AP_LED: track 0.00 -> 47.5 mm, vias 0 -> 2
- net +3V3: track 371.3 -> 326.4 mm, vias 15 -> 14
- net NAV: track 7.33 -> 50.1 mm, vias 0 -> 2
- net BANK: track 7.33 -> 50.1 mm, vias 0 -> 2
- net BC_LED: track 0.00 -> 42.6 mm
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
Commit message: Fully routed!
Connections:
- RN3 pad 5: XFR -> FD2
- RN3 pad 6: YD -> ALT
- RN3 pad 7: ALT -> YD
- RN3 pad 8: /Input shifter1/D0 -> AP
- RN4 pad 5: /Input shifter1/D7 -> XFR
- RN4 pad 7: FD2 -> /Input shifter1/D5
- RN4 pad 8: AP -> /Input shifter1/D4
- U3 pad 10: FD2_LED -> YD_LED
- U3 pad 9: YD_LED -> FD2_LED
- U5 pad 11: /Input shifter1/D0 -> AP
- U5 pad 12: ALT -> YD
- U5 pad 13: YD -> ALT
- U5 pad 14: XFR -> FD2
- U5 pad 3: AP -> /Input shifter1/D4
- U5 pad 4: FD2 -> /Input shifter1/D5
- U5 pad 6: /Input shifter1/D7 -> XFR
Routing:
- net +3V3: track 326.4 -> 395.7 mm, vias 14 -> 22
- net ALT: track 7.33 -> 73.5 mm
- net YD: track 7.33 -> 44.4 mm
- net XFR: track 7.33 -> 44.1 mm
- net FD2: track 7.33 -> 24.8 mm, vias 0 -> 2
- net DISC: track 6.50 -> 22.7 mm
- net AP: track 7.33 -> 20.4 mm
- net FD2_LED: track 78.9 -> 86.3 mm, vias 4 -> 6
- net GND: track 47.1 -> 52.2 mm, vias 31 -> 34
- net VBUS: track 434.0 -> 438.8 mm
- net /Input shifter1/D4: track 0.00 -> 3.88 mm
- net /Input shifter1/D5: track 0.00 -> 3.69 mm
- net /Input shifter/D6: track 0.00 -> 3.33 mm
- net /Input shifter/D5: track 0.00 -> 3.33 mm
- net Net-(R2-Pad1): track 0.00 -> 1.95 mm
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
Commit message: Added 3d models
Other:
- board text added: "JLCJLCJLCJLC"

Commit message: Cleanup based on feedback
Parts:
- moved H14 6.88 mm to (24.1, 59.7)
- moved H13 6.35 mm to (331.5, 22.9)
- moved H1 6.35 mm to (24.1, 17.8)
- moved H12 6.35 mm to (24.1, 23.0)
- moved H2 6.35 mm to (331.5, 17.8)
- moved H3 6.35 mm to (24.1, 64.8)
- moved H4 6.35 mm to (331.5, 64.8)
- moved H10 4.58 mm to (101.9, 25.4)
- moved C13 3.07 mm to (129.6, 35.8)
- moved J3 3.07 mm to (172.6, 61.0)
- moved J4 3.07 mm to (228.5, 61.0)
- moved R4 3.07 mm to (131.1, 50.3)
- moved C16 3.07 mm to (123.6, 44.2)
- moved C19 3.07 mm to (123.3, 37.6)
- moved J1 3.07 mm to (39.3, 61.0)
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Routing:
- net /RP2040/USB_D+: track 12.4 -> 14.8 mm
Other:
- board size 317.5 x 50.8 mm -> 317.5 x 57.1 mm
- board text added: "ALT"
- board text added: "AP"
- board text added: "APPR"
- board text added: "BANK"
- board text added: "BC"
- board text added: "CRS1"
- board text added: "CRS2"
- board text added: "DISC"
- board text added: "FD1"
- board text added: "FD2"
- board text added: "FLC"
- board text added: "HDG"
- board text added: "NAV"
- board text added: "VNAV"
- board text added: "VS"
- board text added: "XFR"
- board text added: "YD"
